File: CAD/AMS2ZWAVE.sch (KiCad schematic (older format))
At the start: 52 parts, among them J1 RJ45_Shielded, J2 Conn_Coaxial, J3 mini simplicity, J4 Conn_01x05_Male, SW1 SW_Push, U1 NCN5150DR2G, U2 LM358, U3 MAX17531AUB+T, U4 ZGM130S

Commit message: PCB iteration 2
* Added inrush current limiter
* Added footprint to use BRD4202 instead of soldering down ZGM130S
Parts:
- added D5: NSI50010, Diode_SMD:D_SOD-123, symbol Device:D_Tunnel
- added J5: BRD_upper, Connector_PinHeader_1.27mm:PinHeader_2x20_P1.27mm_Vertical_SMD, symbol Connector_Generic:Conn_02x20_Odd_Even
- added J6: BRD_lower, Connector_PinHeader_1.27mm:PinHeader_2x20_P1.27mm_Vertical_SMD, symbol Connector_Generic:Conn_02x20_Odd_Even
- C1: value 100n -> 1n
Connections:
- wire segments 245 -> 271
- no-connect marks 36 -> 99
Other:
- note added: "BRD4202A interface"
- moved on the sheet: C13, C14, J2, JP4, U4

Commit message: Update to v2 PCB
* Increased DCDC switching frequency to 600kHz
* Added resistor divider for setting UVLO to 10V
* Added solderjumper for DCDC mode
* Added bulk capacitor to smooth out 12V swings on the input line
Parts:
- added C12: 1n, Capacitor_SMD:C_0805_2012Metric_Pad1.18x1.45mm_HandSolder, symbol Device:C
- added C16: 33u, Capacitor_Tantalum_SMD:CP_EIA-2012-12_Kemet-R_Pad1.30x1.05mm_HandSolder, symbol Device:CP
- added JP8: SolderJumper_2_Open, Jumper:SolderJumper-2_P1.3mm_Open_RoundedPad1.0x1.5mm, symbol Jumper:SolderJumper_2_Open
- added R18: 1M, Resistor_SMD:R_0805_2012Metric_Pad1.20x1.40mm_HandSolder, symbol Device:R
- added R19: 130k, Resistor_SMD:R_0805_2012Metric_Pad1.20x1.40mm_HandSolder, symbol Device:R
- JP1, JP2: footprint Jumper:SolderJumper-2_P1.3mm_Open_RoundedPad1.0x1.5mm -> Jumper:SolderJumper-2_P1.3mm_Bridged_RoundedPad1.0x1.5mm; symbol Jumper:SolderJumper_2_Open -> Jumper:SolderJumper_2_Bridged
- R14: value 140k -> 69.8k
Connections:
- wire segments 271 -> 286
- no-connect marks 99 -> 98
Other:
- moved on the sheet: C5, D4, R14, R15, R16

Commit message: Update to proto v2
* Added edgemount SMA in addition to U.FL for antenna flexibility
Parts:
- added J7: Conn_Coaxial, Connector_Coaxial:SMA_Amphenol_132134-16_Vertical, symbol Connector:Conn_Coaxial
Connections:
- wire segments 286 -> 290
Changed lines of the file:
@@
 U 1 1 6043B78F
 P 7500 5050
-F 0 "J2" H 7428 5288 50  0000 C CNN
-F 1 "Conn_Coaxial" H 7428 5197 50  0000 C CNN
+F 0 "J2" H 7500 5200 50  0000 C CNN
+F 1 "Conn_Coaxial" H 7428 5197 50  0001 C CNN
 F 2 "Connector_Coaxial:U.FL_Molex_MCRF_73412-0110_Vertical" H 7500 5050 50  0001 C CNN
 F 3 " ~" H 7500 5050 50  0001 C CNN
@@
 $EndComp
 Wire Wire Line
-	7500 5250 7500 5400
+	7500 5250 7500 5350
 $Comp
 L power:GND #PWR0126
@@
 $EndComp
 Wire Wire Line
-	7700 5050 8350 5050
+	7700 5050 7850 5050
 Wire Wire Line
 	8350 3150 7850 3150
@@
 Wire Wire Line
 	6500 1400 6550 1400
+$Comp
+L Connector:Conn_Coaxial J7
+U 1 1 60045B35
+P 7850 5350
+F 0 "J7" V 8000 5300 50  0000 L CNN
+F 1 "Conn_Coaxial" V 7823 5450 50  0001 L CNN
+F 2 "Connector_Coaxial:SMA_Amphenol_132134-16_Vertical" H 7850 5350 50  0001 C CNN
+F 3 " ~" H 7850 5350 50  0001 C CNN
+	1    7850 5350
+	0    1    1    0
+$EndComp
+Wire Wire Line
+	7850 5150 7850 5050
+Connection ~ 7850 5050
+Wire Wire Line
+	7850 5050 8350 5050
+Wire Wire Line
+	7650 5350 7500 5350
+Connection ~ 7500 5350
+Wire Wire Line
+	7500 5350 7500 5400
 $EndSCHEMATC

Commit message: Update to proto v2
* Added test points for LGA pads bordering on in-use pads, to avoid them from coming loose when too much heat is applied
* Moved SMA edge connector around, it makes more sense to have it at the top
* Tidied layout
Parts:
- added TP1, TP2, TP3, TP4, TP5, TP6, TP7: TestPoint, TestPoint:TestPoint_THTPad_D1.0mm_Drill0.5mm, symbol Connector:TestPoint
- J7: footprint Connector_Coaxial:SMA_Amphenol_132134-16_Vertical -> Connector_Coaxial:SMA_Samtec_SMA-J-P-X-ST-EM1_EdgeMount
Connections:
- wire segments 290 -> 291
- no-connect marks 98 -> 90
Changed lines of the file:
@@
 Wire Wire Line
 	8350 3250 7850 3250
-NoConn ~ 8350 3550
-NoConn ~ 8350 3450
-NoConn ~ 8350 3350
 NoConn ~ 8350 5350
 NoConn ~ 8350 5450
@@
 NoConn ~ 8350 5750
 NoConn ~ 8350 5850
-NoConn ~ 9950 5850
-NoConn ~ 9950 5550
 NoConn ~ 9950 5450
 NoConn ~ 9950 5350
-NoConn ~ 9950 5250
 NoConn ~ 9950 4650
 NoConn ~ 9950 4550
@@
 NoConn ~ 9950 4250
 NoConn ~ 9950 3650
-NoConn ~ 9950 3250
 NoConn ~ 9950 3150
 NoConn ~ 9950 3050
@@
 Wire Wire Line
 	10150 3750 10150 2850
-NoConn ~ 9950 3450
 Text GLabel 4550 4400 0    50   Input ~ 0
 HAN_TX
@@
 F 0 "J7" V 8000 5300 50  0000 L CNN
 F 1 "Conn_Coaxial" V 7823 5450 50  0001 L CNN
-F 2 "Connector_Coaxial:SMA_Amphenol_132134-16_Vertical" H 7850 5350 50  0001 C CNN
+F 2 "Connector_Coaxial:SMA_Samtec_SMA-J-P-X-ST-EM1_EdgeMount" H 7850 5350 50  0001 C CNN
 F 3 " ~" H 7850 5350 50  0001 C CNN
 	1    7850 5350
@@
 Wire Wire Line
 	7500 5350 7500 5400
+$Comp
+L Connector:TestPoint TP1
+U 1 1 6020C5DE
+P 8350 3350
+F 0 "TP1" V 8350 3700 50  0000 C CNN
+F 1 "TestPoint" V 8454 3422 50  0001 C CNN
+F 2 "TestPoint:TestPoint_THTPad_D1.0mm_Drill0.5mm" H 8550 3350 50  0001 C CNN
+F 3 "~" H 8550 3350 50  0001 C CNN
+	1    8350 3350
+	0    -1   -1   0
+$EndComp
+$Comp
+L Connector:TestPoint TP2
+U 1 1 6020DBC5
+P 8350 3450
+F 0 "TP2" V 8350 3800 50  0000 C CNN
+F 1 "TestPoint" V 8454 3522 50  0001 C CNN
+F 2 "TestPoint:TestPoint_THTPad_D1.0mm_Drill0.5mm" H 8550 3450 50  0001 C CNN
+F 3 "~" H 8550 3450 50  0001 C CNN
+	1    8350 3450
+	0    -1   -1   0
+$EndComp
+$Comp
+L Connector:TestPoint TP3
+U 1 1 6020DE23
+P 8350 3550
+F 0 "TP3" V 8350 3900 50  0000 C CNN
+F 1 "TestPoint" V 8454 3622 50  0001 C CNN
+F 2 "TestPoint:TestPoint_THTPad_D1.0mm_Drill0.5mm" H 8550 3550 50  0001 C CNN
+F 3 "~" H 8550 3550 50  0001 C CNN
+	1    8350 3550
+	0    -1   -1   0
+$EndComp
+$Comp
+L Connector:TestPoint TP5
+U 1 1 60254A15
+P 9950 5850
+F 0 "TP5" V 9950 6200 50  0000 C CNN
+F 1 "TestPoint" V 10054 5922 50  0001 C CNN
+F 2 "TestPoint:TestPoint_THTPad_D1.0mm_Drill0.5mm" H 10150 5850 50  0001 C CNN
+F 3 "~" H 10150 5850 50  0001 C CNN
+	1    9950 5850
+	0    1    1    0
+$EndComp
+$Comp
+L Connector:TestPoint TP4
+U 1 1 6025583D
+P 9950 5550
+F 0 "TP4" V 9950 5900 50  0000 C CNN
+F 1 "TestPoint" V 10054 5622 50  0001 C CNN
+F 2 "TestPoint:TestPoint_THTPad_D1.0mm_Drill0.5mm" H 10150 5550 50  0001 C CNN
+F 3 "~" H 10150 5550 50  0001 C CNN
+	1    9950 5550
+	0    1    1    0
+$EndComp
+Wire Wire Line
+	9950 5250 10150 5250
+$Comp
+L Connector:TestPoint TP7
+U 1 1 602C5F56
+P 9950 3450
+F 0 "TP7" V 10000 3550 50  0000 C CNN
+F 1 "TestPoint" V 10054 3522 50  0001 C CNN
+F 2 "TestPoint:TestPoint_THTPad_D1.0mm_Drill0.5mm" H 10150 3450 50  0001 C CNN
+F 3 "~" H 10150 3450 50  0001 C CNN
+	1    9950 3450
+	0    1    1    0
+$EndComp
+$Comp
+L Connector:TestPoint TP6
+U 1 1 602C710B
+P 9950 3250
+F 0 "TP6" V 9900 3350 50  0000 C CNN
+F 1 "TestPoint" V 10054 3322 50  0001 C CNN
+F 2 "TestPoint:TestPoint_THTPad_D1.0mm_Drill0.5mm" H 10150 3250 50  0001 C CNN
+F 3 "~" H 10150 3250 50  0001 C CNN
+	1    9950 3250
+	0    1    1    0
+$EndComp
 $EndSCHEMATC
